File: nRF52_Sensors/pcb/sensor_tag.sch (EAGLE design)
At the start: 5 parts

Commit message: nRF52 tests ongoing
Parts:
- added U$6: CR2477, cr2477:CR2477
Connections:
- new net RX: U$3.P0_07, U$5.RX
- net GND: now also U$6.GND
- net VCC: now also U$6.VCC
Changed lines of the file:
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@@
 <part name="U$4" library="cr2032" deviceset="CR2032" device=""/>
 <part name="U$5" library="nrf_tag_debug" deviceset="NRF_TAG_DEBUG" device=""/>
+<part name="U$6" library="cr2477" deviceset="CR2477" device=""/>
 </parts>
 <sheets>
@@
 <instance part="U$4" gate="G$1" x="-7.62" y="-5.08"/>
 <instance part="U$5" gate="G$1" x="-68.58" y="0" rot="R180"/>
+<instance part="U$6" gate="G$1" x="33.02" y="-17.78"/>
 </instances>
 <busses>
@@
 <wire x1="-63.5" y1="-5.08" x2="-30.48" y2="-5.08" width="0.1524" layer="91"/>
 <wire x1="-30.48" y1="-5.08" x2="-30.48" y2="-10.16" width="0.1524" layer="91"/>
-<wire x1="-30.48" y1="-10.16" x2="-12.7" y2="-10.16" width="0.1524" layer="91"/>
+<wire x1="-30.48" y1="-10.16" x2="-17.78" y2="-10.16" width="0.1524" layer="91"/>
 <label x="-30.48" y="-10.16" size="1.778" layer="95" rot="R180"/>
+<wire x1="-17.78" y1="-10.16" x2="-12.7" y2="-10.16" width="0.1524" layer="91"/>
+<wire x1="-17.78" y1="-10.16" x2="-17.78" y2="-22.86" width="0.1524" layer="91"/>
+<pinref part="U$6" gate="G$1" pin="GND"/>
+<wire x1="-17.78" y1="-22.86" x2="20.32" y2="-22.86" width="0.1524" layer="91"/>
+<junction x="-17.78" y="-10.16"/>
 </segment>
 <segment>
@@
 <pinref part="U$4" gate="G$1" pin="VCC"/>
 <pinref part="U$5" gate="G$1" pin="VCC"/>
-<wire x1="-12.7" y1="0" x2="-63.5" y2="0" width="0.1524" layer="91"/>
+<wire x1="-12.7" y1="0" x2="-20.32" y2="0" width="0.1524" layer="91"/>
 <label x="-16.002" y="-1.778" size="1.778" layer="95" rot="R180"/>
+<pinref part="U$6" gate="G$1" pin="VCC"/>
+<wire x1="-20.32" y1="0" x2="-63.5" y2="0" width="0.1524" layer="91"/>
+<wire x1="20.32" y1="-12.7" x2="12.7" y2="-12.7" width="0.1524" layer="91"/>
+<wire x1="12.7" y1="-12.7" x2="12.7" y2="7.62" width="0.1524" layer="91"/>
+<wire x1="12.7" y1="7.62" x2="-20.32" y2="7.62" width="0.1524" layer="91"/>
+<wire x1="-20.32" y1="7.62" x2="-20.32" y2="0" width="0.1524" layer="91"/>
+<junction x="-20.32" y="0"/>
 </segment>
 <segment>
@@
 <pinref part="U$3" gate="G$1" pin="P0_06"/>
 <pinref part="U$5" gate="G$1" pin="TX"/>
-<wire x1="-58.42" y1="35.56" x2="-58.42" y2="-10.16" width="0.1524" layer="91"/>
-<wire x1="-58.42" y1="-10.16" x2="-63.5" y2="-10.16" width="0.1524" layer="91"/>
-<label x="-55.88" y="22.606" size="1.778" layer="95"/>
+<wire x1="-58.42" y1="35.56" x2="-58.42" y2="-15.24" width="0.1524" layer="91"/>
+<wire x1="-58.42" y1="-15.24" x2="-63.5" y2="-15.24" width="0.1524" layer="91"/>
+<label x="-60.96" y="22.606" size="1.778" layer="95"/>
 </segment>
 </net>
+<net name="RX" class="0">
+<segment>
+<pinref part="U$3" gate="G$1" pin="P0_07"/>
+<wire x1="-53.34" y1="35.56" x2="-53.34" y2="-10.16" width="0.1524" layer="91"/>
+<pinref part="U$5" gate="G$1" pin="RX"/>
+<wire x1="-53.34" y1="-10.16" x2="-63.5" y2="-10.16" width="0.1524" layer="91"/>
+<label x="-52.324" y="21.082" size="1.778" layer="95"/>
+</segment>
+</net>
